File: PC-370_P2.sch (KiCad schematic (older format))
At the start: 85 parts, among them J1 PC/370-P-M Cable, J2 Bus_ISA_16bit, U1 Conn_02x20_Counter_Clockwise, U10 74LS112, U11 74LS138, U12 74LS138, U13 74S74, U15 74LS20, U16 74LS10, U17 74S00, U18 74S00, U19 74LS175, U2 74LS245, U20 74LS175, U21 74S51, U22 74LS51, U23 74S00, U24 74LS32, U25 74LS245, U26 74LS374, U27 74LS373, U28 74LS374, U29 74LS374, U3 74LS374, U30 74LS244, U31 74S86, U32 74LS20, U33 74LS04, U34 74LS02, U35 74S00, U36 74S74, U37 74S74, U38 74S10, U39 74LS10, U4 74LS374, U40 74S00, U41 74LS02, U42 74LS138, U43 74LS32, U44 74LS153, U45 74LS157, U46 74LS153, U47 74LS153, U48 74S30, U49 74LS00, U5 74LS374, U50 74LS08, U51 74LS30, U52 74LS10, U53 74S09, U54 74LS112, U55 74LS27, U56 IBM_R_Network13_US, U57 74LS04, U58 74LS112, U59 74LS27, U6 74LS245, U60 74LS20, U61 74LS157, U62 74LS244, U63 74LS153, U64 74S157, U66 68000-PGA, U67 68000-PGA, U68 SY2128-1, U69 SY2128-1, U7 74S280, U70 74S241, U71 74LS32, U72 74LS74, U73 74S112, U74 74S112, U75 74LS02, U76 74LS138, U77 74LS125, U78 74LS175, U79 74LS367, U8 74LS02, U80 74LS175, U81 74LS244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

Commit message: Columns 6-8 feeped out.
Connections:
- net A23: now also U49.13
- net Status2_3?: now also U8.4
- net 7-2?_11: now reaches U30.11 (I0b), U30.8 (I3a), U31.11, U49.10, U70.2 (I0a)
- net E_Parity: now reaches U7.5 (Even)
- net E_Parity: now also U31.13
- net 9-2?_6: now reaches U33.6
- net 9-2?_6: now also U49.4
- net 9-2?_8: now reaches U33.8
- net 9-2?_8: now also U23.9, U32.10, U50.5, U52.2
- net 11-2?_6: now reaches U31.1
- net 11-2?_6: now also U35.6
- net at U31.2: now also U31.6
- net at U31.3: now also U31.12
- net 7-3?_8: now reaches U48.8
- net 7-3?_8: now also U38.11
- net at U32.1: now also U8.10
- net 9-1?_6: now reaches U32.4
- net 9-1?_6: now also U10.6 (~Q), U15.10
- net 13-2?_9: now reaches U32.5
- net 13-2?_9: now also U35.2, U37.9 (Q), U38.13
- net 12-2?_5: now reaches U32.12
- net 12-2?_5: now also U10.1 (C), U10.13 (C), U13.4 (~S), U15.12, U17.1, U19.1 (~Mr), U21.13, U35.9, U36.5 (Q), U39.11
- net 8-2?_8: now reaches U32.8
- net 8-2?_8: now also U50.13
- net 9-1?_5: now reaches U32.9
- net 9-1?_5: now also U10.5 (Q), U17.12, U50.4, U55.3
- net 14-4?_4: now reaches U49.2
- net 14-4?_4: now also U16.4, U49.12, U49.9, U61.1 (S), U62.1 (OEa), U75.4
- net at U10.3 (J): now also U8.1
- net at U10.11 (J): now also U8.13
- net 9-1?_9: now reaches U10.9 (Q)
- net 9-1?_9: now also U8.6
- net 11-1?_O6: now reaches U8.3
- net 11-1?_O6: now also U12.9 (O6), U71.2, U8.11
- net 12-1?_5: now reaches U8.5
- net 12-1?_5: now also U13.5 (Q), U15.5, U16.5, U50.10
- no-connect marks 15 -> 19
Changed lines of the file:
@@
 Text Label 11500 17050 0    50   ~ 0
 PB?9
-Wire Wire Line
-	10500 16850 10100 16850
-Wire Wire Line
-	10100 16850 10100 18200
-Connection ~ 10500 16850
 $Comp
 L power:+5V #PWR0131
@@
 	1    0    0    -1
 $EndComp
-Wire Wire Line
-	13350 18200 13350 19900
-Wire Wire Line
-	13350 19900 15200 19900
-Wire Wire Line
-	10100 18200 13350 18200
 Text Notes 12750 23150 0    79   ~ 16
 Page Address Table
@@
 Text Label 26500 12400 2    50   ~ 0
 Status2?_C
-Wire Wire Line
-	13350 18200 13800 18200
-Connection ~ 13350 18200
-Wire Wire Line
-	12900 15250 13350 15250
-Wire Wire Line
-	13350 15250 13350 18200
 Text Label 10500 17350 2    50   ~ 0
 6-2?_OEa
@@
 Text Label 41650 13100 2    50   ~ 0
 A17
+Text Label 11500 13250 0    50   ~ 0
+E_Parity
+Text Label 12300 15350 2    50   ~ 0
+E_Parity
+NoConn ~ 11500 13450
+Wire Wire Line
+	15400 12100 12900 12100
+Wire Wire Line
+	12900 12100 12900 12150
+Wire Wire Line
+	12300 12250 11900 12250
+Wire Wire Line
+	11900 12250 11900 13100
+Wire Wire Line
+	11900 13100 12300 13100
+Text Label 19650 12900 0    50   ~ 0
+11-1?_O6
+Text Label 12300 12250 2    50   ~ 0
+11-1?_O6
+Text Label 17050 19950 2    50   ~ 0
+11-1?_O6
+Text Label 12900 12500 0    50   ~ 0
+Status2_3?
+Text Label 21200 12100 0    50   ~ 0
+12-1?_5
+Text Label 12300 12400 2    50   ~ 0
+12-1?_5
+Text Label 15400 18200 2    50   ~ 0
+12-1?_5
+Text Label 24550 12400 2    50   ~ 0
+12-1?_5
+Text Label 26500 12600 2    50   ~ 0
+12-1?_5
+Text Label 16000 12950 0    50   ~ 0
+9-1?_9
+Text Label 12300 12600 2    50   ~ 0
+9-1?_9
+Wire Wire Line
+	12900 12850 13350 12850
+Wire Wire Line
+	13350 12850 13350 14150
+Wire Wire Line
+	13350 14150 13800 14150
+Wire Wire Line
+	12900 13200 13650 13200
+Wire Wire Line
+	13650 13200 13650 12950
+Wire Wire Line
+	13650 12950 15400 12950
+Text Label 19450 14700 0    50   ~ 0
+11-2?_6
+Text Label 12300 14100 2    50   ~ 0
+11-2?_6
+Wire Wire Line
+	12900 14550 13100 14550
+Wire Wire Line
+	13100 14550 13100 13850
+Wire Wire Line
+	13100 13850 11900 13850
+Wire Wire Line
+	11900 13850 11900 14300
+Wire Wire Line
+	11900 14300 12300 14300
+Wire Wire Line
+	12900 14200 13050 14200
+Wire Wire Line
+	13050 14200 13050 13800
+Wire Wire Line
+	13050 13800 11850 13800
+Wire Wire Line
+	11850 13800 11850 15150
+Wire Wire Line
+	11850 15150 12300 15150
+NoConn ~ 12300 14800
+NoConn ~ 12300 15000
+NoConn ~ 12900 14900
+Text Label 12900 17650 0    50   ~ 0
+7-3?_8
+Text Label 24550 15250 2    50   ~ 0
+7-3?_8
+Text Label 16000 12300 0    50   ~ 0
+9-1?_6
+Text Label 13800 14350 2    50   ~ 0
+9-1?_6
+Text Label 24550 12600 2    50   ~ 0
+9-1?_6
+Text Label 23100 15200 0    50   ~ 0
+13-2?_9
+Text Label 13800 14450 2    50   ~ 0
+13-2?_9
+Text Label 18850 14450 2    50   ~ 0
+13-2?_9
+Text Label 24550 14550 2    50   ~ 0
+13-2?_9
+Text Label 16000 12100 0    50   ~ 0
+9-1?_5
+Text Label 13800 14550 2    50   ~ 0
+9-1?_5
+Text Label 15400 17650 2    50   ~ 0
+9-1?_5
+Text Label 24550 17750 2    50   ~ 0
+9-1?_5
+Text Label 28300 12950 2    50   ~ 0
+9-1?_5
+Text Label 16000 15200 0    50   ~ 0
+9-2?_8
+Text Label 13800 14650 2    50   ~ 0
+9-2?_8
+Text Label 15400 17850 2    50   ~ 0
+9-2?_8
+Text Label 18850 17450 2    50   ~ 0
+9-2?_8
+Text Label 39800 12600 2    50   ~ 0
+9-2?_8
+Text Label 14400 14700 0    50   ~ 0
+8-2?_8
+Text Label 15400 18550 2    50   ~ 0
+8-2?_8
+Text Label 21200 14350 0    50   ~ 0
+12-2?_5
+Text Label 13800 14750 2    50   ~ 0
+12-2?_5
+Text Label 15400 12200 2    50   ~ 0
+12-2?_5
+Text Label 15400 13050 2    50   ~ 0
+12-2?_5
+Text Label 18850 14950 2    50   ~ 0
+12-2?_5
+Text Label 20900 11900 0    50   ~ 0
+12-2?_5
+Text Label 24550 12700 2    50   ~ 0
+12-2?_5
+Text Label 26500 15250 2    50   ~ 0
+12-2?_5
+Text Label 28300 11900 2    50   ~ 0
+12-2?_5
+Text Label 31600 13000 2    50   ~ 0
+12-2?_5
+Text Label 35750 12050 2    50   ~ 0
+12-2?_5
+Wire Wire Line
+	13800 17500 13450 17500
+Wire Wire Line
+	13450 17500 13450 18000
+Wire Wire Line
+	13450 18000 13800 18000
+Wire Wire Line
+	13450 18000 13450 18350
+Wire Wire Line
+	13450 18350 13800 18350
+Connection ~ 13450 18000
+Text Label 25150 20200 0    50   ~ 0
+14-4?_4
+Text Label 13800 17500 2    50   ~ 0
+14-4?_4
+Text Label 26500 12500 2    50   ~ 0
+14-4?_4
+Text Label 35700 18650 2    50   ~ 0
+14-4?_4
+Text Label 37600 18500 2    50   ~ 0
+14-4?_4
+Text Label 16000 14900 0    50   ~ 0
+9-2?_6
+Text Label 13800 17650 2    50   ~ 0
+9-2?_6
+Text Label 12900 15250 0    50   ~ 0
+7-2?_11
+Text Label 10500 16750 2    50   ~ 0
+7-2?_11
+Text Label 13800 18200 2    50   ~ 0
+7-2?_11
+Text Label 15200 19900 2    50   ~ 0
+7-2?_11
+Text Label 13800 18550 2    50   ~ 0
+A23
 $EndSCHEMATC

Commit message: 9-10 done.
Connections:
- net P2J4?: now also U34.9, U76.3 (A2)
- net R-~W: now also U33.3
- net ~AS: now also U33.1, U33.13
- net ~Reset: now also U10.14 (~R), U10.15 (~R), U79.13 (O6b)
- net 15-1?_6: now reaches U70.1 (OEa)
- net 15-1?_6: now also U16.6, U40.5
- net P-UP_12: now reaches U70.4 (I1a)
- net P-UP_12: now also U40.9, U56.12 (R11), U72.10 (~S), U72.13 (~R)
- net 10-4?_6: now reaches U70.6 (I2a)
- net 10-4?_6: now also U71.6
- net 18_1?_6: now reaches U70.8 (I3a)
- net 18_1?_6: now also U19.6 (~Q1)
- net AS_1: now reaches U33.2
- net AS_1: now also U17.10, U36.1 (~R)
- net 15-4?_9: now reaches U33.5
- net 15-4?_9: now also U76.9 (O6)
- net 10-2?_10: now reaches U33.9
- net 10-2?_10: now also U34.10, U34.11, U39.3, U51.11
- net AS_2: now reaches U33.12
- net AS_2: now also U37.1 (~R)
- net 11-4?_6: now reaches U10.2 (K)
- net 11-4?_6: now also U10.12 (K), U72.6 (~Q)
- net P-UP_13: now reaches U10.4 (~S)
- net P-UP_13: now also U10.10 (~S), U54.2 (K), U54.3 (J), U54.4 (~S), U56.13 (R12), U58.10 (~S), U58.4 (~S), U72.1 (~R), U76.6 (E3)
- net 9-1?_7: now reaches U10.7 (~Q)
- net 9-1?_7: now also U39.2
- net A12&A14: now reaches U50.3
- net A12&A14: now also U51.2
- net 9-3?_6: now reaches U50.6
- net 9-3?_6: now also U59.13
- net 9-3?_8: now reaches U50.8
- net 9-3?_8: now also U13.2 (D)
- net 14-2?_8: now reaches U50.9
- net 14-2?_8: now also U38.8
- net 10-1?_7: now reaches U50.12
- net 10-1?_7: now also U11.7 (O7)
- net 10-1?_13: now reaches U11.13 (O2)
- net 10-1?_13: now also U16.13
- net 12-2?_6: now reaches U11.4 (E1)
- net 12-2?_6: now also U12.4 (E1), U34.12, U36.6 (~Q), U37.11 (C), U72.3 (C)
- net 10-3?_8: now reaches U11.5 (E2)
- net 10-3?_8: now also U12.5 (E2), U16.11, U34.2, U51.8, U55.2
- net 10-2?_1: now reaches U34.1
- net 10-2?_1: now also U60.9
- net A13norA15: now reaches U34.4
- net A13norA15: now also U51.12
- net 15_2?_6: now reaches U51.1
- net 15_2?_6: now also U16.10, U39.6, U57.1
- net 10-4?_3: now reaches U71.3
- net 10-4?_3: now also U20.9 (Cp)
- net 18-1?_2: now reaches U71.4
- net 18-1?_2: now also U19.2 (Q0)
- net ~ISA_IOW: now reaches U71.10
- net ~ISA_IOW: now also J2.13 (~IOW), U41.3, U43.5
- net ~PCAMA?_WE: now reaches U71.8
- net ~PCAMA?_WE: now also U83.3 (WE), U84.3 (WE)
- net 18-2?_9: now reaches U71.9
- net 18-2?_9: now also U42.9 (O6), U77.10
- net A23orPAT1_D8: now reaches U71.11
- net A23orPAT1_D8: now also U52.1
- net 11-1?_O6 renamed 11-1?_9
- net ~P-UP_11 renamed P-UP_11
- no-connect marks 19 -> 30
Changed lines of the file:
@@
 NoConn ~ 5850 19450
 Text Label 26600 18350 2    50   ~ 0
-~P-UP_11
+P-UP_11
 Text Label 22800 17950 0    50   ~ 0
-~P-UP_11
+P-UP_11
 Text Label 5850 20550 2    50   ~ 0
-~P-UP_11
+P-UP_11
 Text Label 5850 18950 2    50   ~ 0
-~P-UP_11
+P-UP_11
 NoConn ~ 5850 20350
 NoConn ~ 5850 20450
@@
 Text Label 26500 14550 2    50   ~ 0
 PAT_A-B
-Text Notes 14850 15700 0    300  ~ 60
-*
 Text Label 8800 14250 2    50   ~ 0
 PAT_CE
@@
 Wire Wire Line
 	12900 12100 12900 12150
-Wire Wire Line
-	12300 12250 11900 12250
-Wire Wire Line
-	11900 12250 11900 13100
-Wire Wire Line
-	11900 13100 12300 13100
 Text Label 19650 12900 0    50   ~ 0
-11-1?_O6
+11-1?_9
 Text Label 12300 12250 2    50   ~ 0
-11-1?_O6
+11-1?_9
 Text Label 17050 19950 2    50   ~ 0
-11-1?_O6
+11-1?_9
 Text Label 12900 12500 0    50   ~ 0
 Status2_3?
@@
 Text Label 13800 18550 2    50   ~ 0
 A23
+Wire Wire Line
+	15400 12300 15000 12300
+Wire Wire Line
+	15000 12300 15000 13150
+Wire Wire Line
+	15000 13150 15400 13150
+Text Label 19450 20050 0    50   ~ 0
+11-4?_6
+Text Label 15400 12300 2    50   ~ 0
+11-4?_6
+Wire Wire Line
+	22500 17500 22150 17500
+Wire Wire Line
+	22150 17500 22150 17300
+Wire Wire Line
+	22150 17300 22500 17300
+Wire Wire Line
+	22800 17100 22150 17100
+Wire Wire Line
+	22150 17100 22150 17300
+Connection ~ 22150 17300
+Text Label 26600 18550 2    50   ~ 0
+P-UP_13
+Text Label 30200 17300 0    50   ~ 0
+P-UP_13
+Text Label 30200 18150 0    50   ~ 0
+P-UP_13
+Text Label 26300 20700 2    50   ~ 0
+P-UP_13
+Text Label 22500 17300 2    50   ~ 0
+P-UP_13
+Text Label 19150 20250 0    50   ~ 0
+P-UP_13
+Text Label 15700 11900 0    50   ~ 0
+P-UP_13
+Text Label 15700 12750 0    50   ~ 0
+P-UP_13
+Text Label 16000 13150 0    50   ~ 0
+9-1?_7
+Text Label 26500 14450 2    50   ~ 0
+9-1?_7
+Text Label 15700 12500 0    50   ~ 0
+~Reset
+Text Label 15700 13350 0    50   ~ 0
+~Reset
+Text Label 32650 20700 0    50   ~ 0
+~Reset
+Text Label 15400 14300 2    50   ~ 0
+~AS
+Text Label 15400 15800 2    50   ~ 0
+~AS
+Text Notes 14850 15700 0    300  ~ 60
+*
+Text Label 16000 14300 0    50   ~ 0
+AS_1
+Text Label 20900 14750 0    50   ~ 0
+AS_1
+Text Label 28300 12800 2    50   ~ 0
+AS_1
+Text Label 15400 14600 2    50   ~ 0
+R-~W
+Text Label 15400 14900 2    50   ~ 0
+15-4?_9
+Text Label 17650 15150 0    50   ~ 0
+10-2?_10
+Text Label 17050 15400 2    50   ~ 0
+10-2?_10
+Text Label 15400 15200 2    50   ~ 0
+10-2?_10
+Text Label 17050 18100 2    50   ~ 0
+10-2?_10
+Text Label 26500 14700 2    50   ~ 0
+10-2?_10
+Text Label 16000 15800 0    50   ~ 0
+AS_2
+Text Label 22800 14750 0    50   ~ 0
+AS_2
+Text Label 16000 17400 0    50   ~ 0
+A12&A14
+Text Label 17050 17600 2    50   ~ 0
+A12&A14
+Text Label 16000 17750 0    50   ~ 0
+9-3?_6
+Text Label 31800 17650 2    50   ~ 0
+9-3?_6
+Text Label 25150 15150 0    50   ~ 0
+14-2?_8
+Text Label 15400 18000 2    50   ~ 0
+14-2?_8
+Text Label 16000 18100 0    50   ~ 0
+9-3?_8
+Text Label 20600 12100 2    50   ~ 0
+9-3?_8
+Text Label 17850 13000 0    50   ~ 0
+10-1?_7
+Text Label 27300 20800 0    50   ~ 0
+15-4?_9
+Text Label 15400 18350 2    50   ~ 0
+10-1?_7
+Text Label 12300 13100 2    50   ~ 0
+11-1?_9
+Text Label 26600 18450 2    50   ~ 0
+P-UP_12
+Text Label 28300 15000 2    50   ~ 0
+P-UP_12
+Text Label 15200 20000 2    50   ~ 0
+P-UP_12
+Text Label 19150 20500 0    50   ~ 0
+P-UP_12
+Text Label 19150 21100 0    50   ~ 0
+P-UP_12
+NoConn ~ 16200 20600
+NoConn ~ 16200 20500
+Text Label 17650 20200 0    50   ~ 0
+10-4?_6
+Text Label 15200 20100 2    50   ~ 0
+10-4?_6
+Text Label 32600 12400 0    50   ~ 0
+18_1?_6
+Text Label 15200 20200 2    50   ~ 0
+18_1?_6
+NoConn ~ 16200 20400
+NoConn ~ 16200 20300
+NoConn ~ 15200 20300
+NoConn ~ 15200 20400
+NoConn ~ 15200 20500
+NoConn ~ 15200 20600
+Text Label 27100 12500 0    50   ~ 0
+15-1?_6
+Text Label 15200 20800 2    50   ~ 0
+15-1?_6
+Text Label 28300 14850 2    50   ~ 0
+15-1?_6
+NoConn ~ 15200 20900
+Text Label 21200 14550 0    50   ~ 0
+12-2?_6
+Text Label 16850 13000 2    50   ~ 0
+12-2?_6
+Text Label 18650 13000 2    50   ~ 0
+12-2?_6
+Text Label 17050 15600 2    50   ~ 0
+12-2?_6
+Text Label 18850 19950 2    50   ~ 0
+12-2?_6
+Text Label 22500 15300 2    50   ~ 0
+12-2?_6
+Text Label 17650 17800 0    50   ~ 0
+10-3?_8
+Text Label 16850 12900 2    50   ~ 0
+10-3?_8
+Text Label 17050 14350 2    50   ~ 0
+10-3?_8
+Text Label 18650 12900 2    50   ~ 0
+10-3?_8
+Text Label 24550 17500 2    50   ~ 0
+10-3?_8
+Text Label 26500 12950 2    50   ~ 0
+10-3?_8
+NoConn ~ 17850 12900
+Text Label 17850 12500 0    50   ~ 0
+10-1?_13
+Text Label 26500 12250 2    50   ~ 0
+10-1?_13
+NoConn ~ 17850 12300
+Text Label 17650 14450 0    50   ~ 0
+10-2?_1
+Text Label 33850 18000 2    50   ~ 0
+10-2?_1
+Text Label 17650 14800 0    50   ~ 0
+A13norA15
+Text Label 17050 18200 2    50   ~ 0
+A13norA15
+Text Label 17050 15250 2    50   ~ 0
+P2J4?
+Text Label 26300 20400 2    50   ~ 0
+P2J4?
+Text Label 27100 14800 0    50   ~ 0
+15_2?_6
+Text Label 28300 17300 2    50   ~ 0
+15_2?_6
+Text Label 17050 17500 2    50   ~ 0
+15_2?_6
+Text Label 26500 12850 2    50   ~ 0
+15_2?_6
+Text Label 17650 19850 0    50   ~ 0
+10-4?_3
+Text Label 33650 12900 2    50   ~ 0
+10-4?_3
+Text Label 32600 12100 0    50   ~ 0
+18-1?_2
+Text Label 17050 20100 2    50   ~ 0
+18-1?_2
+Text Label 17650 20550 0    50   ~ 0
+~PCAMA?_WE
+Text Label 40550 20800 0    50   ~ 0
+~PCAMA?_WE
+Text Label 42400 20800 0    50   ~ 0
+~PCAMA?_WE
+Text Label 32600 15050 0    50   ~ 0
+18-2?_9
+Text Label 17050 20450 2    50   ~ 0
+18-2?_9
+Text Label 28600 21250 0    50   ~ 0
+18-2?_9
+Entry Wire Line
+	24750 22850 24850 22950
+Text Label 43900 26400 2    50   ~ 0
+~ISA_IOW
+Text Label 17050 20650 2    50   ~ 0
+~ISA_IOW
+Text Label 29900 14500 2    50   ~ 0
+~ISA_IOW
+Text Label 33850 14700 2    50   ~ 0
+~ISA_IOW
+Text Label 17650 20900 0    50   ~ 0
+A23orPAT1_D8
+Text Label 18850 17350 2    50   ~ 0
+A23orPAT1_D8
 $EndSCHEMATC

Commit message: 11-13 done.
Connections:
- net Clk1: now also U13.3 (C), U73.12 (K)
- net DB_A-B: now also U12.6 (E3)
- net GND: now also U54.12 (K)
- net Status2_7?: now also U52.12
- net M-Cable_49: now reaches J1.49 (Pin_49)
- net M-Cable_49: now also U73.13 (C)
- net PAT2_D1norD2: now reaches U31.2, U31.6
- net 7-2?_3: now reaches U31.12, U31.3
- net 11-1?_13: now reaches U12.13 (O2)
- net 11-1?_13: now also U17.4
- net 11-1?_14: now reaches U12.14 (O1)
- net 11-1?_14: now also U41.11, U41.5
- net 11-1?_7: now reaches U12.7 (O7)
- net 11-1?_7: now also U72.2 (D)
- net 12-1?_6: now reaches U35.1
- net 12-1?_6: now also U13.6 (~Q), U21.2, U38.1, U59.2
- net 11-2?_3: now reaches U35.3
- net 11-2?_3: now also U13.12 (D)
- net 11-2?_11: now reaches U35.10
- net 11-2?_11: now also U35.11
- net 11-2?_8: now reaches U35.8
- net 11-2?_8: now also U53.1, U53.13, U54.1 (C)
- net 14-2?_12: now reaches U35.13
- net 14-2?_12: now also U38.12
- net 19-1?_10: now reaches U52.13
- net 19-1?_10: now also U20.10 (Q2), U75.6
- net Clk1_Lt'd_FPU_Busy: now reaches U52.3
- net Clk1_Lt'd_FPU_Busy: now also U52.9, U72.8 (~Q)
- net ~Status_Lt'd_FPU_Ready: now reaches U52.5
- net ~Status_Lt'd_FPU_Ready: now also U54.7 (~Q)
- net 11-3?_6: now reaches U52.6
- net 11-3?_6: now also U59.5
- net 11-3?_8: now reaches U52.8
- net 11-3?_8: now also U75.3
- net P-UP_8: now reaches U13.1 (~R)
- net P-UP_8: now also U13.10 (~S), U13.13 (~R), U56.8 (R7)
- net 14-3?_8: now reaches U36.2 (D)
- net 14-3?_8: now also U38.4, U55.8
- net P-UP_10: now reaches U36.4 (~S)
- net P-UP_10: now also U36.10 (~S), U37.4 (~S), U56.10 (R9)
- net AS_3: now reaches U36.13 (~R)
- net AS_3: now also U18.1, U40.12, U40.2, U40.8, U54.14 (~R)
- net ~Clk1_Lt'd_AB_HL_C: now reaches U36.8 (~Q)
- net ~Clk1_Lt'd_AB_HL_C: now also U38.9
- net Clk1_Lt'd_AB_HL_C: now reaches U36.9 (Q)
- net Clk1_Lt'd_AB_HL_C: now also U17.13, U19.9 (Cp), U37.2 (D)
- net P-UP_6: now reaches U37.10 (~S)
- net P-UP_6: now also U56.6 (R5), U73.15 (~R), U73.4 (~S)
- net 13-3?_5: now reaches U37.12 (D)
- net 13-3?_5: now also U53.5, U54.5 (Q)
- net 13-2?_8: now reaches U37.8 (~Q)
- net 13-2?_8: now also U18.9, U39.4
- net 19-4?_7: now reaches U53.2
- net 19-4?_7: now also U53.12, U80.7 (Q1), U81.4 (I1a)
- net 13-3?_6: now reaches U53.9
- net 13-3?_6: now also U54.6 (~Q)
- net 18-4?_7: now reaches U73.1 (C)
- net 18-4?_7: now also U74.1 (C), U74.13 (C), U79.7 (O3a)
- net at U73.2 (K): now also U73.5 (Q)
- net at U73.3 (J): now also U73.6 (~Q)
- net P-UP_9: now reaches U73.10 (~S)
- net P-UP_9: now also U56.9 (R8), U73.14 (~R), U74.15 (~R)
- net Status_Lt'd_FPU_Ready: now reaches U54.9 (Q)
- net Status_Lt'd_FPU_Ready: now also U55.5
- net 13-4?_5: now reaches U74.2 (K)
- net 13-4?_5: now also U74.12 (K), U74.5 (Q)
- net 13-4?_9: now reaches U74.3 (J)
- net 13-4?_9: now also U74.9 (Q)
- net P-UP_5: now reaches U74.4 (~S)
- net P-UP_5: now also U56.5 (R4), U74.10 (~S), U74.14 (~R)
- no-connect marks 30 -> 39
Other:
- note added: "Clock Divider"
- note added: "Proccessor Bus Grant Ack"
