File: PC-370_P2.sch (KiCad schematic (older format))
At the start: 85 parts, among them J1 PC/370-P-M Cable, J2 Bus_ISA_16bit, U1 Conn_02x20_Counter_Clockwise, U10 74LS112, U11 74LS138, U12 74LS138, U13 74S74, U15 74LS20, U16 74LS10, U17 74S00, U18 74S00, U19 74LS175, U2 74LS245, U20 74LS175, U21 74S51, U22 74LS51, U23 74S00, U24 74LS32, U25 74LS245, U26 74LS374, U27 74LS373, U28 74LS374, U29 74LS374, U3 74LS374, U30 74LS244, U31 74S86, U32 74LS20, U33 74LS04, U34 74LS02, U35 74S00, U36 74S74, U37 74S74, U38 74S10, U39 74LS10, U4 74LS374, U40 74S00, U41 74LS02, U42 74LS138, U43 74LS32, U44 74LS153, U45 74LS157, U46 74LS153, U47 74LS153, U48 74S30, U49 74LS00, U5 74LS374, U50 74LS08, U51 74LS30, U52 74LS10, U53 74S09, U54 74LS112, U55 74LS27, U56 IBM_R_Network13_US, U57 74LS04, U58 74LS112, U59 74LS27, U6 74LS245, U60 74LS20, U61 74LS157, U62 74LS244, U63 74LS153, U64 74S157, U66 68000-PGA, U67 68000-PGA, U68 SY2128-1, U69 SY2128-1, U7 74S280, U70 74S241, U71 74LS32, U72 74LS74, U73 74S112, U74 74S112, U75 74LS02, U76 74LS138, U77 74LS125, U78 74LS175, U79 74LS367, U8 74LS02, U80 74LS175, U81 74LS244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

Commit message: Minor corrections made, and columns 14-16 done.
Connections:
- net 12-2?_5: now also U39.1
- net 9-1?_7: now also U38.2; no longer U39.2
- net FC0: now also U76.1 (A0)
- net FC1: now also U76.2 (A1)
- net GND: now also U76.4 (E1), U76.5 (E2), U77.9
- net PB?0: no longer U21.4
- net ~DB_CE: now also U15.13, U57.10; no longer U55.10
- net M-Cable_37: now reaches J1.37 (Pin_37)
- net M-Cable_37: now also U22.3, U44.2 (S1), U46.2 (S1), U47.2 (S1), U57.3, U63.2 (S1), U64.1 (S)
- net M-Cable_43: now reaches J1.43 (Pin_43)
- net M-Cable_43: now also U75.8
- net 14-2?_6: now reaches J1.45 (Pin_45)
- net 14-2?_6: now also U38.6
- net 14-1?_6: now reaches U15.6
- net 14-1?_6: now also U17.5
- net 14-1?_8: now reaches U15.8
- net 14-1?_8: now also U16.1, U16.2
- net 18-3?_12: now reaches U38.5
- net 18-3?_12: now also U59.12
- net 14-3?_12: now reaches U55.12
- net 14-3?_12: now also U55.11
- net 14-4?_13: now reaches U55.13
- net 14-4?_13: now also U75.13
- net 15-4?_12: now reaches U55.4
- net 15-4?_12: now also U18.12, U22.13, U57.11, U76.12 (O3)
- net 14-3?_6: now reaches U55.6
- net 14-3?_6: now also U55.10
- net 14-4?_1: now reaches U75.1
- net 14-4?_1: now also U75.12
- net 22-1?_8: now reaches U75.5
- net 22-1?_8: now also U23.8, U24.1, U24.5, U24.9
- net 10-4?_10: now reaches U75.10
- net 10-4?_10: now also U78.1 (~Mr), U80.1 (~Mr)
- net ISA_RESET: now reaches U75.9
- net ISA_RESET: now also J2.2 (RESET)
- net 18-3?_6: now reaches U75.11
- net 18-3?_6: now also U59.6
- net 15-1?_12: now reaches U16.12
- net 15-1?_12: now also U18.5
- net 15-1?_8: now reaches U16.8
- net 15-1?_8: now also U21.1, U59.1
- net 16-1?_11: now reaches U16.9
- net 16-1?_11: now also U17.11
- net 16-3?_2: now reaches U39.9
- net 16-3?_2: now also U17.2, U39.2, U57.2
- net 15-4?_10: now reaches U76.10 (O5)
- net 15-4?_10: now also U22.12, U57.5
- net 16-1?_6: now reaches U17.6
- net 16-1?_6: now also U17.9
- net 16-2?_6: now reaches U40.1
- net 16-2?_6: now also U40.6
- net 16-3?_8: now reaches U40.13
- net 16-3?_8: now also U57.8
- net ~M-Cable_37: now reaches U57.4
- net ~M-Cable_37: now also U21.4
- net 16-3?_6: now reaches U57.6
- net 16-3?_6: now also U22.10, U22.11
- net ISA_REFRESH: now reaches U57.12
- net ISA_REFRESH: now also U21.5, U23.1
- net ~ISA_REFRESH: now reaches U57.13
- net ~ISA_REFRESH: now also J2.19 (~REFRESH), U23.12
- net 19-4?_11: now reaches U77.1
- net 19-4?_11: now also U80.11 (~Q2)
- net IRQ7: now reaches U77.3
- net IRQ7: now also J2.21 (IRQ7)
- net 19-2?_8: now reaches U77.4
- net 19-2?_8: now also U43.8
- net P1_IPL1: now reaches U77.5
- net P1_IPL1: now also U58.9 (Q)
- net ISA_DB7: now reaches U77.6
- net ISA_DB7: now also J2.33 (DB7)
- net ~ISA_IOCS16: now reaches U77.8
- net ~ISA_IOCS16: now also J2.64 (~IOCS16)
- net ISA_DB4: now reaches U77.11
- net ISA_DB4: now also J2.36 (DB4), U78.4 (D0), U84.4 (D1)
- net 17_4?_2: now reaches U77.12
- net 17_4?_2: now also U78.2 (Q0)
- net 19-2?_3: now reaches U77.13
- net 19-2?_3: now also U43.3, U81.1 (OEa)
- net P1J4? renamed P2_FC2
- net P2J4? renamed P1_FC2
- no-connect marks 39 -> 45
Other:
- note added: "P1 FC Decode"
- note added: "Supervisor Data"
- note added: "Supervisor Prog"
- note added: "Undef Reserved"

Commit message: Added 74S51 part to AT370 library, its different from an LS51! Finished beeping out the rest of the board! The current schematic will be archived and re-aranging and re-labeling of nets will begin.
Parts:
- U21: symbol 74xx:74LS51 -> AT370:74S51
Connections:
- net 12-1?_6: now also U18.10
- net 14-4?_4: now also U45.1 (S); no longer U62.1 (OEa)
- net 22-1?_8: now also U24.12
- net AS_3: now also U18.4
- net GND: now also U44.1 (Ea), U44.15 (Eb), U45.15 (E), U46.1 (Ea), U46.15 (Eb), U47.1 (Ea), U47.15 (Eb), U61.15 (E), U62.11 (I0b), U62.8 (I3a), U63.1 (Ea), U63.15 (Eb), U64.15 (E), U79.1 (OEa), U79.15 (OEb), U81.11 (I0b), U81.13 (I1b), U81.15 (I2b), U81.17 (I3b), U82.15 (E)
- net M-Cable_37: now also U21.3; no longer U22.3
- net Status2_7?: no longer U35.12
- net ~ISA_IOW: now also U41.9
- net M-Cable_2: now reaches J1.2 (Pin_2)
- net M-Cable_2: now also U47.7 (Za)
- net M-Cable_28: now reaches J1.28 (Pin_28)
- net M-Cable_28: now also U64.4 (Za)
- net M-Cable_29: now reaches J1.29 (Pin_29)
- net M-Cable_29: now also U64.7 (Zb)
- net M-Cable_3: now reaches J1.3 (Pin_3)
- net M-Cable_3: now also U47.9 (Zb)
- net M-Cable_31: now reaches J1.31 (Pin_31)
- net M-Cable_31: now also U64.9 (Zc)
- net M-Cable_32: now reaches J1.32 (Pin_32)
- net M-Cable_32: now also U64.12 (Zd)
- net M-Cable_35: now reaches J1.35 (Pin_35)
- net M-Cable_35: now also U21.10, U21.9
- net M-Cable_39: now reaches J1.39 (Pin_39)
- net M-Cable_39: now also U44.14 (S0), U46.14 (S0), U47.14 (S0), U63.14 (S0)
- net M-Cable_4: now reaches J1.4 (Pin_4)
- net M-Cable_4: now also U46.7 (Za)
- net 20-1?_6: now reaches J1.41 (Pin_41)
- net 20-1?_6: now also U21.6
- net 18-2?_12: now reaches J1.47 (Pin_47)
- net 18-2?_12: now also U42.12 (O3)
- net M-Cable_5: now reaches J1.5 (Pin_5)
- net M-Cable_5: now also U46.9 (Zb)
- net M-Cable_6: now reaches J1.6 (Pin_6)
- net M-Cable_6: now also U63.7 (Za)
- net M-Cable_7: now reaches J1.7 (Pin_7)
- net M-Cable_7: now also U63.9 (Zb)
- net M-Cable_8: now reaches J1.8 (Pin_8)
- net M-Cable_8: now also U44.7 (Za)
- net M-Cable_9: now reaches J1.9 (Pin_9)
- net M-Cable_9: now also U44.9 (Zb)
- net ~ISA_IOR: now reaches J2.14 (~IOR)
- net ~ISA_IOR: now also U43.12, U43.2, U43.9
- net ISA_CLK: now reaches J2.20 (CLK)
- net ISA_CLK: now also U79.12 (I5)
- net ISA_OSC: now reaches J2.30 (OSC)
- net ISA_OSC: now also U79.6 (I3)
- net ISA_DB6: now reaches J2.34 (DB6)
- net ISA_DB6: now also U84.10 (D3)
- net ISA_DB5: now reaches J2.35 (DB5)
- net ISA_DB5: now also U84.6 (D2)
- net ISA_DB3: now reaches J2.37 (DB3)
- net ISA_DB3: now also U80.13 (D3), U81.12 (O3a), U81.9 (O0b), U83.10 (D3)
- net ISA_DB2: now reaches J2.38 (DB2)
- net ISA_DB2: now also U80.12 (D2), U81.14 (O2a), U81.7 (O1b), U83.6 (D2)
- net ISA_DB1: now reaches J2.39 (DB1)
- net ISA_DB1: now also U80.5 (D1), U81.16 (O1a), U81.5 (O2b), U83.4 (D1)
- net ISA_DB0: now reaches J2.40 (DB0)
- net ISA_DB0: now also U80.4 (D0), U81.18 (O0a), U81.3 (O3b)
- net ISA_AEN: now reaches J2.42 (AEN)
- net ISA_AEN: now also U42.4 (E1)
- net ISA_BA16: now reaches J2.46 (BA16)
- net ISA_BA16: now also U62.6 (I2a), U82.13 (I1d)
- net ISA_BA15: now reaches J2.47 (BA15)
- net ISA_BA15: now also U62.13 (I1b), U82.10 (I1c)
- net ISA_BA14: now reaches J2.48 (BA14)
- net ISA_BA14: now also U62.4 (I1a), U82.6 (I1b)
- net ISA_BA13: now reaches J2.49 (BA13)
- net ISA_BA13: now also U62.15 (I2b), U82.3 (I1a)
- net ISA_BA12: now reaches J2.50 (BA12)
- net ISA_BA12: now also U46.10 (I0b)
- net ISA_BA11: now reaches J2.51 (BA11)
- net ISA_BA11: now also U46.6 (I0a)
- net ISA_BA10: now reaches J2.52 (BA10)
- net ISA_BA10: now also U47.10 (I0b)
- net ISA_BA09: now reaches J2.53 (BA09)
- net ISA_BA09: now also U47.6 (I0a), U60.1
- net ISA_BA08: now reaches J2.54 (BA08)
- net ISA_BA08: now also U23.13, U60.2
- net ISA_BA07: now reaches J2.55 (BA07)
- net ISA_BA07: now also U44.11 (I1b), U59.9
- net ISA_BA06: now reaches J2.56 (BA06)
- net ISA_BA06: now also U59.10, U63.11 (I1b)
- net ISA_BA05: now reaches J2.57 (BA05)
- net ISA_BA05: now also U60.4, U63.5 (I1a)
- net ISA_BA04: now reaches J2.58 (BA04)
- net ISA_BA04: now also U46.11 (I1b), U60.5
- net ISA_BA03: now reaches J2.59 (BA03)
- net ISA_BA03: now also U46.5 (I1a), U59.11
- net ISA_BA02: now reaches J2.60 (BA02)
- net ISA_BA02: now also U42.3 (A2), U47.11 (I1b)
- net ISA_BA01: now reaches J2.61 (BA01)
- net ISA_BA01: now also U42.2 (A1), U47.5 (I1a)
- net ISA_BA00: now reaches J2.62 (BA00)
- net ISA_BA00: now also U79.4 (I2)
- net ISA_SBHE: now reaches J2.81 (SBHE)
- net ISA_SBHE: now also U79.10 (I4)
- net ISA_DB12: now reaches J2.95 (D12)
- net ISA_DB12: now also U82.2 (I0a)
- net ISA_DB13: now reaches J2.96 (D13)
- net ISA_DB13: now also U82.5 (I0b)
- net ISA_DB14: now reaches J2.97 (D14)
- net ISA_DB14: now also U82.11 (I0c)
- net ISA_DB15: now reaches J2.98 (D15)
- net ISA_DB15: now also U82.14 (I0d)
- net 17-2?_1: now reaches U41.1
- net 17-2?_1: now also U58.2 (K)
- net 18-2?_11: now reaches U41.2
- net 18-2?_11: now also U42.11 (O4)
- net 17-2?_4: now reaches U41.4
- net 17-2?_4: now also U58.3 (J)
- net 17-2?_10: now reaches U41.10
- net 17-2?_10: now also U58.11 (J)
- net 18-2?_13: now reaches U41.8
- net 18-2?_13: now also U42.13 (O2), U43.10
- net 17-2?_13: now reaches U41.13
- net 17-2?_13: now also U58.12 (K)
- net 18-4?_11: now reaches U58.1 (C)
- net 18-4?_11: now also U58.13 (C), U79.11 (O5b)
- net 17-4?_3: now reaches U78.3 (~Q0)
- net 17-4?_3: now also U82.1 (S)
- net 19-2?_6: now reaches U78.9 (Cp)
- net 19-2?_6: now also U43.6, U80.9 (Cp)
- net 18-1?_7: now reaches U19.7 (Q1)
- net 18-1?_7: now also U70.8 (I3a)
- net 18-4?_5: now reaches U42.1 (A0)
- net 18-4?_5: now also U23.2, U64.11 (I0c), U79.5 (O2a)
- net 18-2?_14: now reaches U42.14 (O1)
- net 18-2?_14: now also U43.1, U43.4
- net 18-2?_15: now reaches U42.15 (O0)
- net 18-2?_15: now also U43.13
- net 19-3?_6: now reaches U42.5 (E2)
- net 19-3?_6: now also U60.6
- net 18-3?_8: now reaches U42.6 (E3)
- net 18-3?_8: now also U59.8
- net 19-1?_2: now reaches U20.2 (Q0)
- net 19-1?_2: now also U22.1
- net 19-1?_7: now reaches U20.7 (Q1)
- net 19-1?_7: now also U22.9
- net 19-4?_2: now reaches U79.14 (I6)
- net 19-4?_2: now also U80.2 (Q0), U81.2 (I0a)
- net 18-4?_9: now reaches U79.9 (O4a)
- net 18-4?_9: now also U64.14 (I0d)
- net 19-4?_10: now reaches U80.10 (Q2)
- net 19-4?_10: now also U81.6 (I2a)
- net ~PCAMA?_CS: now reaches U80.14 (~Q3)
- net ~PCAMA?_CS: now also U83.2 (CS), U84.2 (CS)
- net 19-4?_15: now reaches U80.15 (Q3)
- net 19-4?_15: now also U62.1 (OEa), U62.19 (OEb), U81.8 (I3a)
- net 19-2?_11: now reaches U43.11
- net 19-2?_11: now also U81.19 (OEb)
- net 19-3?_8: now reaches U60.8
- net 19-3?_8: now also U35.12
- net 21-3?_12: now reaches U62.12 (O3a)
- net 21-3?_12: now also U64.5 (I0b), U84.9 (O3)
- net 21-3?_14: now reaches U62.14 (O2a)
- net 21-3?_14: now also U44.10 (I0b), U84.5 (O1)
- net 21-3?_16: now reaches U62.16 (O1a)
- net 21-3?_16: now also U63.10 (I0b), U83.7 (O2)
- net 21-3?_5: now reaches U62.5 (O2b)
- net 21-3?_5: now also U63.6 (I0a), U83.5 (O1)
- net 21-3?_7: now reaches U62.7 (O1b)
- net 21-3?_7: now also U44.6 (I0a), U83.9 (O3)
- net 21-3?_9: now reaches U62.9 (O0b)
- net 21-3?_9: now also U64.2 (I0a), U84.7 (O2)
- net 20-3?_12: now reaches U61.12 (Zd)
- net 20-3?_12: now also U46.12 (I2b)
- net 23-1?_8: now reaches U61.2 (I0a)
- net 23-1?_8: now also U24.8
- net 20-3?_4: now reaches U61.4 (Za)
- net 20-3?_4: now also U44.4 (I2a)
- net 20-3?_7: now reaches U61.7 (Zb)
- net 20-3?_7: now also U63.12 (I2b)
- net 20-3?_9: now reaches U61.9 (Zc)
- net 20-3?_9: now also U63.4 (I2a)
- net PCAMA_A3: now reaches U82.12 (Zd)
- net PCAMA_A3: now also U83.13 (A3), U84.13 (A3)
- net PCAMA_A0: now reaches U82.4 (Za)
- net PCAMA_A0: now also U83.1 (A0), U84.1 (A0)
- net PCAMA_A1: now reaches U82.7 (Zb)
- net PCAMA_A1: now also U83.15 (A1), U84.15 (A1)
- net PCAMA_A2: now reaches U82.9 (Zc)
- net PCAMA_A2: now also U83.14 (A2), U84.14 (A2)
- net 23-1?_11: now reaches U45.11 (I0c)
- net 23-1?_11: now also U24.11
- net 21-2?_12: now reaches U45.12 (Zd)
- net 21-2?_12: now also U44.12 (I2b)
- net 23-1?_3: now reaches U45.14 (I0d)
- net 23-1?_3: now also U24.3
- net 23-1?_6: now reaches U45.5 (I0b)
- net 23-1?_6: now also U24.6
- net 21-2?_7: now reaches U45.7 (Zb)
- net 21-2?_7: now also U64.6 (I1b)
- net 21-2?_9: now reaches U45.9 (Zc)
- net 21-2?_9: now also U64.3 (I1a)
- net 22-1?_6: now reaches U44.5 (I1a)
- net 22-1?_6: now also U23.6
- net 21-1?_8: now reaches U22.8
- net 21-1?_8: now also U23.10
- net 22-1?_3: now reaches U23.3
- net 22-1?_3: now also U23.5
- net 22-1?_11: now reaches U23.4
- net 22-1?_11: now also U23.11
- net 18_1?_6: no longer names the net of U19.6 (~Q1)
- net 18_1?_6: no longer U70.8 (I3a)
- no-connect marks 45 -> 90
Other:
- note added: "Note: 74S51 has two missing inputs compared to 74LS51"
- moved on the sheet: U18A, U18B, U18C, U18D, U41A, U41B, U41C, U41D, U58A, U58B, U78

Commit message: Begin organizing gates, relabeling nets, and general documentation. PCAMA and I/O Regs 0x330-0x337 started.
Connections:
- net 18-2?_13: no longer U42.13 (O2), U43.10
- net 13-4?_5: no longer names the net of U74.12 (K), U74.2 (K), U74.5 (Q)
- net 13-4?_9: no longer names the net of U74.3 (J), U74.9 (Q)
- net 17-2?_1: no longer names the net of U41.1, U58.2 (K)
- net 17-2?_10: no longer names the net of U41.10, U58.11 (J)
- net 17-2?_13: no longer names the net of U41.13, U58.12 (K)
- net 17-2?_4: no longer names the net of U41.4, U58.3 (J)
- net 18-2?_11 renamed ~IOA_334
- net 18-2?_12 renamed ~IOA_333
- net 18-2?_14 renamed ~IOA_331
- net 18-2?_15 renamed ~IOA_330
- net 18-2?_9 renamed ~IOA_336
- net 18-3?_8: no longer names the net of U42.6 (E3), U59.8
- net 18-4?_11 renamed ISA_CLK_Drv
- net 18-4?_5 renamed ISA_BA00_Drv
- net 18-4?_7 renamed ISA_OSC_Drv
- net 18-4?_9 renamed ISA_SBHE_Drv
- net 19-2?_11 renamed ~IOR_330
- net 19-2?_3 renamed ~IOR_331
- net 19-2?_6 renamed ~IOW_331
- net 19-2?_8 renamed ~IOR_332
- net 19-3?_6: no longer names the net of U42.5 (E2), U60.6
- net 21-3?_12 renamed MSA18
- net 21-3?_14 renamed MSA16
- net 21-3?_16 renamed MSA14
- net 21-3?_5 renamed MSA13
- net 21-3?_7 renamed MSA15
- net 21-3?_9 renamed MSA17
- net CLK2 renamed CLK_4.77
- net ~PCAMA?_CS renamed ~PCAMA_CS
- net ~PCAMA?_WE renamed ~PCAMA_WE
- new net ~IOA_332: U42.13 (O2), U43.10
Other:
- note added: "16 x 8 bit\nPCAMA"
- note added: "Address\nDecode"
- note added: "B\ni\nt\ns\n\n1\n7\n\nt\no\n\n1\n9"
- note added: "Divide by 3\n14.318 Mhz / 3 = 4.77 Mhz"
- note added: "Enabled when D3\nis equal to 0."
- note added: "Enabled when D3\nis equal to 1."
- note added: "I/O Reg X'366' Write"
- note added: "I/O Register Decode\nX'330' to X'337'"
- note added: "M\nS\nA\n\nB\ni\nt\ns\n\n1\n3\n\nt\no\n\n1\n8"
- note added: "On PC/370-M2 Board"
- note added: "Operation Register\nRead I/O Reg X'330'/X'331'"
- note added: "Operation Register\nWrite I/O Reg X'331'"
- note added: "PC Address Bus\nPCA00 to PCA19"
- note added: "PCA00 to\nPCA12"
- note added: "PCAMA\nAT/370 Technical Reference\nPage 2-16"
- note added: "P\nC\nA\n\nB\ni\nt\ns\n\n1\n3\n\nt\no\n\n1\n6"
- note added: "S/370 Storage Access Control"
- note added: "Tri-State\nDriver"
- moved on the sheet: J2, R2, U41A, U41B, U41C, U41D, U43A, U43B, U43C, U43D, U44, U45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

Commit message: I/O Registers completely mostly. Started piecing together PAT.
Connections:
- net 18-2?_13 is gone; now on net ~IOA_332: U41.8
- net 10-2?_1: no longer names the net of U34.1, U60.9
- net 10-4?_10 renamed ~Reset_Op_Reg
- net 11-2?_8: no longer names the net of U35.8, U53.1, U53.13, U54.1 (C)
- net 11-3?_6: no longer names the net of U52.6, U59.5
- net 11-3?_8: no longer names the net of U52.8, U75.3
- net 13-3?_5: no longer names the net of U37.12 (D), U53.5, U54.5 (Q)
- net 13-3?_6: no longer names the net of U53.9, U54.6 (~Q)
- net 14-3?_12: no longer names the net of U55.11, U55.12
- net 14-3?_6: no longer names the net of U55.10, U55.6
- net 14-4?_1: no longer names the net of U75.1, U75.12
- net 14-4?_13: no longer names the net of U55.13, U75.13
- net 15-4?_12 renamed DB_CE
- net 16-2?_6: no longer names the net of U40.1, U40.6
- net 16-3?_8: no longer names the net of U40.13, U57.8
- net 17-4?_3 renamed ~OpReg_4
- net 17_4?_2 renamed OpReg_4
- net 18-3?_6: no longer names the net of U59.6, U75.11
- net 19-4?_10 renamed OpReg_2
- net 19-4?_11 renamed ~OpReg_2
- net 19-4?_15 renamed OpReg_3
- net 19-4?_2 renamed OpReg_0
- net 19-4?_7 renamed OpReg_1
- net 23-1?_11: no longer names the net of U24.11, U45.11 (I0c)
- net 23-1?_3: no longer names the net of U24.3, U45.14 (I0d)
- net 23-1?_6: no longer names the net of U24.6, U45.5 (I0b)
- net 23-1?_8: no longer names the net of U24.8, U61.2 (I0a)
- net FPU_15? renamed ~OpReg_0
- net P1_IPL1 renamed 370_INT_07
- net PAT1_WE renamed ~PAT1_WE
- net PAT2_WE renamed ~PAT2_WE
- net Status_3? renamed PCINT_07
- net ~IOR_330: no longer names the net of U43.11, U81.19 (OEb)
- net ~IOR_331: no longer names the net of U43.3, U77.13, U81.1 (OEa)
- net ~IOR_332: no longer names the net of U43.8, U77.4
- net ~IOW_331: no longer names the net of U43.6, U78.9 (Cp), U80.9 (Cp)
- net ~P1_IPL1 renamed ~370_INT_07
- net ~PCAMA_CS renamed ~OpReg_3
Other:
- note added: "Address Translate Mode Reg?\nPatent No: 4,714,993\nFig. 2"
- note added: "Bit 0: ~Enable~/Disable Reset\nBit 1: ~Enable~/Disable Proc 1 & 2 Halt\nBit 2: Enable/~Disable~ IRQ7\nBit 3: Enable/~Disable~ PCAMA\nBit 4: Enable/~Disable~ Write PCAMA"
- note added: "Halt Circuitry"
- note added: "Hardware ID Reg\nRead I/O Reg X'330'\nRead as zeros from bit 0-3"
- note added: "I/O Reg X'366' Write 16-bit"
- note added: "Mux\nPatent No: 4,714,993\nFig. 2"
- note added: "Operation Register\nRead I/O Reg X'331'"
- note added: "PC Diagnostic Parity Control Register\nRead/Write I/O Reg X'333' Circuitry on P/370-M2 board."
- note added: "PC Interrupt Request Register\nWrite I/O Reg X'334' to Clear"
- note added: "PC to PC/370 Address Mapping Register\nAT/370 Technical Reference\nPage 2-13"
- note added: "PC/370 Interrupt Request Register\nWrite I/O Reg X'332' to Set\nRead I/O Reg X'332' to Check\nBit 7: Pending/~Not Pending~ Interrupt from PC AT"
- note added: "PCIB_IN must be set at control store address X'6050'\nAT/370 Technical Reference\nPage 2-9"
- note added: "PCIB_OUT will be set at control store X'6054'\nAT/370 Technical Reference\nPage 2-11"
- note added: "Reset"
- note removed: "I/O Reg X'366' Write"
- note removed: "Operation Register\nRead I/O Reg X'330'/X'331'"
- moved on the sheet: R2, U16B, U17A, U24A, U24B, U24C, U24D, U30, U34A, U35C, U37B, U39A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

Commit message: Logic paths roughly laid out... Some notes added.
Connections:
- net 10-2?_10 renamed User_Space
- net 14-1?_6: no longer names the net of U15.6, U17.5
- net 14-1?_8: no longer names the net of U15.8, U16.1, U16.2
- net 15-1?_12: no longer names the net of U16.12, U18.5
- net 16-1?_6: no longer names the net of U17.6, U17.9
- net 9-2?_8 renamed ~User_Space
- net AB_HL_C renamed Address_Latch_Clock
- net Clk1_Lt'd_AB_HL_C renamed Clk1_Lt'd_Address_Latch_Clock
- net DB_A-B renamed ~R~-W
- net DB_CE renamed FPU_~Data~-Command
- net PAT1_D1 renamed PA12
- net PAT1_D2 renamed PA13
- net PAT1_D3 renamed PA14
- net PAT1_D4 renamed PA15
- net PAT1_D5 renamed PA16
- net PAT1_D6 renamed PA17
- net PAT1_D7 renamed PA18
- net PAT_A-B renamed R-~W~_2
- net ~Clk1_Lt'd_AB_HL_C renamed ~Clk1_Lt'd_Address_Latch_Clock
- net ~DB_CE renamed FPU_Data-~Command
Other:
- note added: "* Relinquishes Reset at the beginning\nof a bus cycle when ~AS~ goes low."
- note added: "FPU Address A8-A15 Decode 5FXX?"
- note added: "FPU addressed 5F2X (hex) range\nPatent No: 4,814,977\nCol 6 Row 35"
- note added: "FPU/Reg? Read Decode"
- note added: "FPU/Reg? Write Decode"
- note added: "Proccessor 1/2 Bus Grant\nAck Interlock"
- note added: "Storage Selection Override Reg\nPatent No: 4,591,982\nFig. 2 OL1/OL2"
- note removed: "Proccessor Bus Grant Ack"
- moved on the sheet: R2, U1, U10C, U13A, U13B, U13C, U15A, U15B, U15C, U16A, U16C, U16D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

Commit message: Major Clean-up. Things roughly laid out near connecting logic... Need to dig into patents and figure out logical chunks and draw out bus cycles to figure out logic.
Connections:
- net Status_LE renamed ~Clk1
Other:
- note added: "Mystery FPU\nHeavily modified 287XL?"
- note added: "System Clock Divider\n16Mhz / 2 ?"
- note removed: "10"
- note removed: "11"
- note removed: "12"
- note removed: "13"
- note removed: "14"
- note removed: "15"
- note removed: "16"
- note removed: "17"
- note removed: "18"
- note removed: "19"
- note removed: "20"
- note removed: "21"
- note removed: "22"
- note removed: "23"
- note removed: "4"
- note removed: "5"
- note removed: "6"
- note removed: "7"
- note removed: "8"
- note removed: "9"
- note removed: "Mystery FPU\nHeavily modified 287?"
- moved on the sheet: J1, J2, R1, R2, U1, U10A, U10B, U11, U12, U13A, U13B, U15A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

Commit message: Storage Selection Override identified and labeled, from patent 4,591,982.
Connections:
- net 10-4?_3: no longer names the net of U20.9 (Cp), U71.3
- net 15-4?_10 renamed ~Operand_Access
- net 15-4?_9 renamed ~Instruction_Fetch
- net 16-3?_6 renamed Operand_Access
- net 19-1?_2 renamed Instr_Override_Latch
- net 19-1?_7 renamed Oper_Override_Latch
- net 21-1?_8 renamed ~CS_Address_Override
- net 22-1?_8 renamed CS_Address_Override
Other:
- note added: "Control Storage Address Override\nPatent No: 4,591,982\nFig. 2 Item: 20"
- note added: "Hardware Registers Address A8-A15 Decode 5FXX?"
- note added: "If !UserSpace or A23=0 or"
- note added: "Proccessor Switch Latch\nPatent No: 4,591,982\nFig. 2"
- note added: "Processor 2 Selected out of POR"
- note removed: "FPU Address A8-A15 Decode 5FXX?"
- note removed: "Proccessor 1/2 Bus Grant\nAck Interlock"
- moved on the sheet: U11, U12, U17A, U22A, U23C, U24A, U24B, U24C, U24D, U27, U45, U57C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

Commit message: More progress, address decoding for memory mapped registers 5FXX being slowly labeled.
Connections:
- net 10-1?_13 renamed ~Read_FPU
- net 11-1?_13 renamed ~Write_FPU
- net 7-1?_1: no longer names the net of U10.3 (J), U8.1
- net 7-1?_13: no longer names the net of U10.11 (J), U8.13
- net Status2?_OE renamed ~Read_BER_REG
- net Status_OE renamed ~Read_CC_INT_REG
- net ~AB_H_OE renamed ~Read_ADDR_REG_High
- net ~AB_L_OE renamed ~Read_ADDR_REG_Low
Other:
- note added: ""QUATCH/OBATCH"\nOp Code Register\nReturn Code Register\n5F7X/5FFX"
- note added: "5F22/5FA2 Command\n5F20/5FA0 Data"
- note added: "A1 used to toggle between Command/Data\nPatent No: 4,814,977\nCol 7 Row 15"
- note added: "Both A1 and FPU_~Data~-Command\nmust be high to select Command from FPU"
- note added: "Bus Error Register 5F3X/5FBX\nBER_REG"
- note added: "CC_INT_REG Register 5F1X/5F9X\nBit 15: PCINT_07\nBit 14-10: Unused\nBit 9: ~370_INT_07~\nBit 8: ~P1_IPL0~\nBit 7: ~FPU_Busy~\nBit 6: FPU_Ready\nBit 5-2: Unused\nBit 1: FPU_CC1\nBit 0: FPU_CC0"
- note added: "CKM"
- note added: "CLK"
- note added: "CMD0"
- note added: "CMD1"
- note added: "D0"
- note added: "D1"
- note added: "D10"
- note added: "D11"
- note added: "D12"
- note added: "D13"
- note added: "D14"
- note added: "D15"
- note added: "D2"
- note added: "D3"
- note added: "D4"
- note added: "D5"
- note added: "D6"
- note added: "D7"
- note added: "D8"
- note added: "D9"
- note added: "FPU addressed 5F2X/5FAX\nPatent No: 4,814,977\nCol 6 Row 35"
- note added: "Meanings? From source code:\nBUS ERROR SUBROUTINE"
- note added: "Mystery FPU\nHeavily modified 287XL?\n287XL pinout if die rotated\n180 Degrees in blue"
- note added: "N.C."
- note added: "NPS2"
- note added: "Odd Program Counter"
- note added: "PAT Parity Error"
- note added: "PEREQ"
- note added: "Page Fault"
- note added: "Real Address Out of Bounds"
- note added: "SYS_CNTL Register 5F2X/5FEX\nBit 0: Instruction Control Store Override Latch\nBit 1: Operand Control Store Override Latch\nBit 2: Bypass PAT bit to access Low Store"
- note added: "VCC"
- note added: "VSS"
- note added: "Virtual Address Out of Bounds"
- note added: "~Busy"
- note added: "~Error"
- note added: "~NPRD"
- note added: "~NPS1"
- note added: "~NPWR"
- note added: "~PEACK"
- note removed: "Mystery FPU\nHeavily modified 287XL?"
- moved on the sheet: R2, U2, U25, U27, U74A, U74B
