File: PC-370_P2.sch (KiCad schematic (older format))
At the start: 85 parts, among them J1 PC/370-P-M Cable, J2 Bus_ISA_16bit, U1 Conn_02x20_Counter_Clockwise, U10 74LS112, U11 74LS138, U12 74LS138, U13 74S74, U15 74LS20, U16 74LS10, U17 74S00, U18 74S00, U19 74LS175, U2 74LS245, U20 74LS175, U21 74S51, U22 74LS51, U23 74S00, U24 74LS32, U25 74LS245, U26 74LS374, U27 74LS373, U28 74LS374, U29 74LS374, U3 74LS374, U30 74LS244, U31 74S86, U32 74LS20, U33 74LS04, U34 74LS02, U35 74S00, U36 74S74, U37 74S74, U38 74S10, U39 74LS10, U4 74LS374, U40 74S00, U41 74LS02, U42 74LS138, U43 74LS32, U44 74LS153, U45 74LS157, U46 74LS153, U47 74LS153, U48 74S30, U49 74LS00, U5 74LS374, U50 74LS08, U51 74LS30, U52 74LS10, U53 74S09, U54 74LS112, U55 74LS27, U56 IBM_R_Network13_US, U57 74LS04, U58 74LS112, U59 74LS27, U6 74LS245, U60 74LS20, U61 74LS157, U62 74LS244, U63 74LS153, U64 74S157, U66 68000-PGA, U67 68000-PGA, U68 SY2128-1, U69 SY2128-1, U7 74S280, U70 74S241, U71 74LS32, U72 74LS74, U73 74S112, U74 74S112, U75 74LS02, U76 74LS138, U77 74LS125, U78 74LS175, U79 74LS367, U8 74LS02, U80 74LS175, U81 74LS244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

Commit message: Lots of net names added, BER_REG labeled, OBATCH reg documented, SYS_CNTL reg documented, some of bus error trigger latch documented.
Connections:
- net 10-1?_7 renamed ~Read_OBATCH
- net 11-1?_14 renamed ~Write_INTR_REG
- net 11-1?_7 renamed ~Write_ENGINE_A
- net 11-1?_9 renamed ~Write_SYS_CNTL
- net 11-2?_3: no longer names the net of U13.12 (D), U35.3
- net 12-1?_5 renamed No_Bus_Error
- net 12-1?_6 renamed Bus_Error
- net 13-2?_8 renamed Proc2_Active
- net 13-2?_9 renamed Proc1_Active
- net 14-2?_8: no longer names the net of U38.8, U50.9
- net 14-4?_4 renamed ~Bypass_PAT
- net 19-1?_10 renamed Bypass_PAT
- net 22-1?_11: no longer names the net of U23.11, U23.4
- net 22-1?_3: no longer names the net of U23.3, U23.5
- net 22-1?_6: no longer names the net of U23.6, U44.5 (I1a)
- net 7-3?_8 renamed Any_Bus_Err
- net 9-2?_6 renamed Instruction_Fetch
- net 9-3?_8: no longer names the net of U13.2 (D), U50.8
- net PB?B_C renamed OBATCH_Clock
- net PB?B_OE renamed ~OBATCH_OE
- net Status2?_C renamed Clock_BER_REG
- net Status2_13? renamed ~Page_Fault
- net Status2_14? renamed ~PAT_Parity_Err
- net Status2_17? renamed ~Off_Boundry
- net Status2_18? renamed ~Virt_Addr_Out_of_Bounds
- net Status2_4? renamed ~Odd_Program_Counter
- net Status2_7? renamed ~Real_Addr_Out_of_Bounds
Other:
- note added: "ADDR_REG\nStores failing 370 address on a bus error."
- note added: "BAGIT Bit\nActive Low\nForce Bus Error to A-Engine"
- note added: "Bus Error Latch\nResets to 1."
- note added: "FPU/Reg Read Decode"
- note added: "FPU/Reg Write Decode"
- note added: "Latches at the end of ANY write cycle\nwhen AS goes low.\nSo when we write to 57FX/5FFX to\nswitch between processors the RC\nwill get stored here."
- note added: "Meanings From source code:\n"BUS ERROR SUBROUTINE"\n"PRIORITY OF HANDLING A-ENGINE BUS ERRORS""
- note added: "Off Boundry"
- note added: "Off-Boundry Bit\nActive Low\nA-Engine will re-run bus cycle"
- note added: "SYS_CNTL Register 5F2X/5FEX\nBit 0: Instruction Control Store Override Latch\nBit 1: Operand Control Store Override Latch\nBit 2: Bypass PAT bit to access Low Store\nBit 4: Off-Boundry Bit\nBit 5: BAGIT Bit"
- note added: "Write to 5FXX"
- note added: "~Read~/Write"
- note added: "~Write to 5F7X/5FFX"
- note removed: "FPU/Reg? Read Decode"
- note removed: "FPU/Reg? Write Decode"
- note removed: "Meanings? From source code:\nBUS ERROR SUBROUTINE"
- note removed: "SYS_CNTL Register 5F2X/5FEX\nBit 0: Instruction Control Store Override Latch\nBit 1: Operand Control Store Override Latch\nBit 2: Bypass PAT bit to access Low Store"
- moved on the sheet: U10A, U10B, U13A, U13B, U17A, U18A, U18C, U19, U21B, U22A, U23C, U32A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

Commit message: PAT Parity Gen/Check info added thanks to help from TubeTime.
Connections:
- net 11-2?_6: no longer names the net of U31.1, U35.6
- net 7-2?_11 renamed PAT_Parity
- net 7-2?_3: no longer names the net of U31.12, U31.3
- net 9-1?_5 renamed Off-Boundry_Bit
- net 9-1?_6 renamed ~Off-Boundry_Bit
- net 9-1?_7 renamed ~BAGIT_Bit
- net 9-1?_9 renamed BAGIT_Bit
- net PAT2_D1xorD2: no longer names the net of U31.2, U31.6
- net PAT2_D4 renamed PA_Parity
- net Status_Lt'd_FPU_Ready renamed ~Clk1~_Lt'd_FPU_Ready
- net User_Space renamed Control_Store
- net ~Status_Lt'd_FPU_Ready renamed ~Clk1~_~Lt'd_FPU_Ready~
- net ~User_Space renamed ~Control_Store
Other:
- note added: "0 When:\nFPU_Busy, !FPU_Ready, 5FA0\nFPU_Busy, FPU_Ready, 5F92\nFPU_Busy, !FPU_Ready, 5F92\nOR\n!Off-Boundry_Bit, FPU_Data, or !FPU_Ready"
- note added: "As soon as a bus error is hit we\ntrigger the BERR pin of the active\nprocessor to handle the error."
- note added: "BAGIT Bit\nWrite 0 to latch.\nForce Bus Error to A-Engine"
- note added: "Goes low when a Proc_Switch is requested\ntoggles back high to latch the Proc Switch\nLatch when bus cycle concludes."
- note added: "Off-Boundry Bit\nWrite 0 to latch.\nA-Engine will re-run bus cycle"
- note added: "PAT Parity Generator/Check"
- note added: "PA_Parity is the parity bit stored in the PAT memory.\nThe NAND gate prevents it from summing into the parity\nduring a write, and it is only summed in during a read.\nWhich verifies the parity with the PA_Parity bit stored."
- note added: "Proc_Switch"
- note added: "SYS_CNTL Register 5F2X/5FEX\nBit 0: Instruction Control Store Override Latch\nBit 1: Operand Control Store Override Latch\nBit 2: Bypass PAT bit to access Low Store\nBit 4: ~Off-Boundry Bit~\nBit 5: ~BAGIT Bit~"
- note added: "U30 gates "PAT_Parity" (the parity output) so that\nit appears on PA_Parity during a write to the PAT memory."
- note added: "~5FXX and ControlStore and (!Proc2_Active or A23=0)"
- note added: "~Off-Boundry Set or FPU Command or FPU_Ready"
- note removed: "BAGIT Bit\nActive Low\nForce Bus Error to A-Engine"
- note removed: "FPU addressed 5F2X (hex) range\nPatent No: 4,814,977\nCol 6 Row 35"
- note removed: "If !UserSpace or A23=0 or"
- note removed: "Off-Boundry Bit\nActive Low\nA-Engine will re-run bus cycle"
- note removed: "SYS_CNTL Register 5F2X/5FEX\nBit 0: Instruction Control Store Override Latch\nBit 1: Operand Control Store Override Latch\nBit 2: Bypass PAT bit to access Low Store\nBit 4: Off-Boundry Bit\nBit 5: BAGIT Bit"
- moved on the sheet: U16B, U16C, U17D, U19, U21A, U31A, U31B, U31D, U33D, U35B, U38B, U39A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
